File: moisture-sensor-carrier.kicad_pcb (KiCad board)
At the start: 4 copper layers, 42 x 155 mm, 61 parts, among them J1 USB-C receptacle, J2 Battery - Adafruit 1578, J3 Solar panel, J4 SWD 10p 1.27mm, J5 U.FL-R-SMT-1(10) antenna, U1 nRF54L15-QFAA, U2 nPM1300-QEAA, U3 FDC1004, U4 SHT45-AD1F, U5 TPS7A1650 5V LDO, X1 CM8V-T1A 32.768kHz CL=7pF 20p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, X2 FA-128 32MHz CL=8pF

Commit message: Baseline before the schematic redraw and layout audit
Nudge C25 and rotate it -90. The schematic and project file changes are
KiCad 10's re-save: property blocks gain show_name/do_not_autoplace and
the s-expressions get pretty-printed. No netlist change.

Co-Authored-By: Claude Opus 5 <noreply@anthropic.com>
Parts:
- moved R21 3.65 mm to (72.1, 100.6), turned to -90 degrees
- moved C25 3.42 mm to (69.2, 100.6), turned to -90 degrees
Routing:
- net /VSET1: track 0.00 -> 2.32 mm
- net /+3V3: track 41.5 -> 40.5 mm, vias 19 -> 18
- net GND: vias 139 -> 138
Changed lines of the file:
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@@
 	(footprint "Capacitor_SMD:C_0402_1005Metric_Pad0.74x0.62mm_HandSolder"
 		(layer "F.Cu")
-		(at 72.5 101.5)
+		(at 69.2 100.6 -90)
 		(descr "Capacitor SMD 0402 (1005 Metric), square (rectangular) end terminal, IPC-7351 nominal with elongated pad for handsoldering. (Body size source: IPC-SM-782 page 76, https://www.pcb-3d.com/wordpress/wp-content/uploads/ipc-sm-782a_amendment_1_and_2.pdf)")
 		(tags "capacitor handsolder")
 		(property "Reference" "C25"
-			(at 0 -1.16 0)
+			(at 0 -1.16 90)
 			(layer "F.Fab")
 			(effects
@@
 		)
 		(property "Value" "100nF X5R"
-			(at 0 1.16 0)
+			(at 0 1.16 90)
 			(layer "F.Fab")
 			(effects
@@
 		)
 		(property "Datasheet" ""
-			(at 0 0 0)
+			(at 0 0 90)
 			(layer "F.Fab")
 			(hide yes)
@@
 		)
 		(property "Description" ""
-			(at 0 0 0)
+			(at 0 0 90)
 			(layer "F.Fab")
 			(hide yes)
@@
 		)
 		(property "KiLib_Generator" "SMD_2terminal_chip_molded"
-			(at 0 0 0)
+			(at 0 0 90)
 			(layer "F.SilkS")
 			(hide yes)
@@
 		(duplicate_pad_numbers_are_jumpers no)
 		(fp_line
-			(start -0.115835 -0.36)
-			(end 0.115835 -0.36)
+			(start -0.115835 0.36)
+			(end 0.115835 0.36)
 			(stroke
 				(width 0.12)
@@
 		)
 		(fp_line
-			(start -0.115835 0.36)
-			(end 0.115835 0.36)
+			(start -0.115835 -0.36)
+			(end 0.115835 -0.36)
 			(stroke
 				(width 0.12)
@@
 		)
 		(fp_text user "${REFERENCE}"
-			(at 0 0 0)
+			(at 0 0 90)
 			(layer "F.Fab")
 			(effects
@@
 		)
 		(pad "1" smd roundrect
-			(at -0.5675 0)
+			(at -0.5675 0 270)
 			(size 0.735 0.62)
 			(layers "F.Cu" "F.Mask" "F.Paste")
@@
 		)
 		(pad "2" smd roundrect
-			(at 0.5675 0)
+			(at 0.5675 0 270)
 			(size 0.735 0.62)
 			(layers "F.Cu" "F.Mask" "F.Paste")
@@
 	(footprint "Resistor_SMD:R_0402_1005Metric_Pad0.72x0.64mm_HandSolder"
 		(layer "F.Cu")
-		(at 68.5 100)
+		(at 72.1 100.6 -90)
 		(descr "Resistor SMD 0402 (1005 Metric), square (rectangular) end terminal, IPC-7351 nominal with elongated pad for handsoldering. (Body size source: IPC-SM-782 page 72, https://www.pcb-3d.com/wordpress/wp-content/uploads/ipc-sm-782a_amendment_1_and_2.pdf)")
 		(tags "resistor handsolder")
 		(property "Reference" "R21"
-			(at 0 -1.17 0)
+			(at 0 -1.17 90)
 			(layer "F.Fab")
 			(effects
@@
 		)
 		(property "Value" "0R disables BUCK1"
-			(at 0 1.17 0)
+			(at 0 1.17 90)
 			(layer "F.Fab")
 			(effects
@@
 		)
 		(property "Datasheet" ""
-			(at 0 0 0)
+			(at 0 0 90)
 			(layer "F.Fab")
 			(hide yes)
@@
 		)
 		(property "Description" ""
-			(at 0 0 0)
+			(at 0 0 90)
 			(layer "F.Fab")
 			(hide yes)
@@
 		)
 		(property "KiLib_Generator" "SMD_2terminal_chip_molded"
-			(at 0 0 0)
+			(at 0 0 90)
 			(layer "F.SilkS")
 			(hide yes)
@@
 		(duplicate_pad_numbers_are_jumpers no)
 		(fp_line
-			(start -0.167621 -0.38)
-			(end 0.167621 -0.38)
+			(start -0.167621 0.38)
+			(end 0.167621 0.38)
 			(stroke
 				(width 0.12)
@@
 		)
 		(fp_line
-			(start -0.167621 0.38)
-			(end 0.167621 0.38)
+			(start -0.167621 -0.38)
+			(end 0.167621 -0.38)
 			(stroke
 				(width 0.12)
@@
 		)
 		(fp_text user "${REFERENCE}"
-			(at 0 0 0)
+			(at 0 0 90)
 			(layer "F.Fab")
 			(effects
@@
 		)
 		(pad "1" smd roundrect
-			(at -0.5975 0)
+			(at -0.5975 0 270)
 			(size 0.715 0.64)
 			(layers "F.Cu" "F.Mask" "F.Paste")
@@
 		)
 		(pad "2" smd roundrect
-			(at 0.5975 0)
+			(at 0.5975 0 270)
 			(size 0.715 0.64)
 			(layers "F.Cu" "F.Mask" "F.Paste")
@@
 	)
 	(via
-		(at 71.5 100)
-		(size 0.6)
-		(drill 0.3)
-		(layers "F.Cu" "B.Cu")
-		(net "GND")
-	)
-	(via
 		(at 78.8 64.8)
 		(size 0.6)
@@
 	)
 	(segment
-		(start 71.9325 101.5)
-		(end 71.93 102.5)
-		(width 0.4)
-		(layer "F.Cu")
-		(net "/+3V3")
-	)
-	(segment
 		(start 79.921 61.6)
 		(end 80.7 61.6)
@@
 	)
 	(via
-		(at 71.93 102.5)
-		(size 0.6)
-		(drill 0.3)
-		(layers "F.Cu" "B.Cu")
-		(net "/+3V3")
-	)
-	(via
 		(at 82.4 75)
 		(size 0.6)
@@
 	)
 	(segment
+		(start 72.1 100.0025)
+		(end 72.1 97.924299)
+		(width 0.2)
+		(layer "F.Cu")
+		(net "/VSET1")
+	)
+	(segment
+		(start 72.1 97.924299)
+		(end 71.9257 97.749999)
+		(width 0.2)
+		(layer "F.Cu")
+		(net "/VSET1")
+	)
+	(segment

Commit message: Draw every rail as a power symbol instead of a text label
+3V3 appeared 21 times as plain text, and VSYS, VBAT, VBUS_IN, SOLAR_PANEL,
SOLAR_5V and FDC_VDD the same way. A label is only a name: one typo in one
copy splits the rail in two and ERC has no reason to object. A power symbol
is checked as a rail and reads as one. Text labels drop 146 -> 94, and the
36 that remain are signals, which is what labels are for.

KiCad ships +3V3 and GND but none of the rest, so tools_gen_power_lib.py
generates them into lib/power_local.kicad_sym -- supply rails drawn as a bar,
derived and gated rails as an open arrow.

Power symbols are global, so those seven nets lose the root-sheet slash:
"/VBAT" becomes "VBAT". Everything keyed on the old spelling had to follow, and
none of it would have failed loudly:

  - seven netclass_patterns in the .kicad_pro would have quietly stopped
    matching, dropping Power width and clearance on the whole supply
  - the DRU charge-path rule went the same way as the A.Net bug already
    recorded in its comment: parses, matches nothing, never fires
  - tools_dru_test.py injects on /VBAT, which is what caught it -- 18/19

Also drop the /RF_C netclass pattern. No such net exists.

Add tools_netcmp.py, which fingerprints the netlist so a redraw can be proven
to have changed drawing only. It reports this commit as identical: 101 nets,
same nodes. DRU 19/19, DRC unchanged at 9 violations and 44 unconnected.

Co-Authored-By: Claude Opus 5 <noreply@anthropic.com>
Connections:
- net /+3V3 renamed +3V3
- net /FDC_VDD renamed FDC_VDD
- net /SOLAR_5V renamed SOLAR_5V
- net /SOLAR_PANEL renamed SOLAR_PANEL
- net /VBAT renamed VBAT
- net /VBUS_IN renamed VBUS_IN
- net /VSYS renamed VSYS
