File: moisture-sensor-carrier.kicad_pcb (KiCad board)
At the start: 4 copper layers, 42 x 155 mm, 43 parts, among them J4 SWD 10p 1.27mm, J5 U.FL-R-SMT-1(10) antenna, U1 nRF54L15-QFAA, U2 nPM2100-QEAA, U3 FDC1004, U4 SHT45-AD1F, X1 CM8V-T1A 32.768kHz CL=7pF 20p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, X2 FA-128 32MHz CL=8pF

Commit message: chore: checkpoint current hardware design and review work
Parts:
- removed C1, C2: 2.2uF/2.5V X6T, Capacitor_SMD:C_0402_1005Metric_Pad0.74x0.62mm_HandSolder
- removed C10, C4, C7, C8: 100nF X7R, Capacitor_SMD:C_0402_1005Metric_Pad0.74x0.62mm_HandSolder
- removed C11: 0.3pF C0G, Capacitor_SMD:C_0201_0603Metric
- removed C12: 10nF/6.3V X7R, Capacitor_SMD:C_0402_1005Metric_Pad0.74x0.62mm_HandSolder
- removed C5: 2.2nF X7R, Capacitor_SMD:C_0402_1005Metric_Pad0.74x0.62mm_HandSolder
- removed C6: 1.5pF, Capacitor_SMD:C_0201_0603Metric
- removed C9: 2.0pF, Capacitor_SMD:C_0201_0603Metric
- removed FB1: FB 120R@100MHz, Inductor_SMD:L_0402_1005Metric_Pad0.77x0.64mm_HandSolder
- removed J5: U.FL-R-SMT-1(10) antenna, Connector_Coaxial:U.FL_Hirose_U.FL-R-SMT-1_Vertical
- removed L1: 4.7uH, Inductor_SMD:L_0603_1608Metric_Pad1.05x0.95mm_HandSolder
- removed L2: 2.7nH, Inductor_SMD:L_0201_0603Metric
- removed L3, L4: 3.5nH, Inductor_SMD:L_0201_0603Metric
- removed NT1: GND_PA to GND (under U1, F.Cu), footprints:NetTie_VSSPA
- removed NT2: GND_C9 to GND (B.Cu only), NetTie:NetTie-2_SMD_Pad0.5mm
- removed X2: FA-128 32MHz CL=8pF, footprints:XTAL_FA-128_2016_4Pin
- added C28: 100nF 16V X7R, Capacitor_SMD:C_0402_1005Metric, F.Cu at (0.00, 0.00)
- added D1, D2, D3: TPD1E1B04DPYR, footprints:TI_DPY0002A, F.Cu at (0.00, 0.00)
- added D10, D4, D5, D6, D7, D8, D9: TPD1E01B04DPYR, footprints:TI_DPY0002A, F.Cu at (0.00, 0.00)
- added FID1, FID2, FID3 (x2): Fiducial, Fiducial:Fiducial_0.5mm_Mask1mm, F.Cu at (0.00, 0.00)
- added Q1: DMG2305UX-7, Package_TO_SOT_SMD:SOT-23, F.Cu at (0.00, 0.00)
- added R30, R31: 5.1k 1%, Resistor_SMD:R_0402_1005Metric, F.Cu at (0.00, 0.00)
- added R32, R33, R34, R35: 100 1%, Resistor_SMD:R_0402_1005Metric, F.Cu at (0.00, 0.00)
- added REF**: LayerMarker_4_6.35x2.54mm_TextH1mm_P1.27mm, Symbol:LayerMarker_4_6.35x2.54mm_TextH1mm_P1.27mm, F.Cu at (0.00, 0.00)
- BT1: value BU2032SM-BT-GTR -> CR2032-BS-6; footprint footprints:BatteryHolder_MPD_BU2032SM-BT-GTR -> footprints:BatteryHolder_LianXin_CR2032-BS-6
- C13: footprint Capacitor_SMD:C_0402_1005Metric_Pad0.74x0.62mm_HandSolder -> Capacitor_SMD:C_0402_1005Metric
- C22, C24: value 1nF X5R -> 1nF 50V X7R; footprint Capacitor_SMD:C_0201_0603Metric -> Capacitor_SMD:C_0402_1005Metric
- C26: value 1uF/10V X7R -> 1uF 10V X7R
- C27: value 100nF X7R -> 100nF 16V X7R; footprint Capacitor_SMD:C_0402_1005Metric_Pad0.74x0.62mm_HandSolder -> Capacitor_SMD:C_0402_1005Metric
- C3: value 10uF/6.3V X6S 0402 -> 10uF/16V X6S; footprint Capacitor_SMD:C_0603_1608Metric_Pad1.08x0.95mm_HandSolder -> Capacitor_SMD:C_0603_1608Metric
- R1: footprint Resistor_SMD:R_0402_1005Metric_Pad0.72x0.64mm_HandSolder -> Resistor_SMD:R_0402_1005Metric
- U1: value nRF54L15-QFAA -> 453-00001R BL54L15; footprint footprints:QFN48_6X6_NOR -> footprints:Ezurio_BL54L15_453-00001
Connections:
- net FDC_VDD renamed +3V3_FDC_SW
- BT1 pad 1: VBAT -> /VBAT_RAW
- J4 pad 10: /SWD_RST -> /RESET_EXT
- J4 pad 2: /SWDIO -> /SWDIO_EXT
- J4 pad 4: /SWDCLK -> /SWDCLK_EXT
- J4 pad 6: /P2.07_SWO -> /SWO_EXT
- L10 pad 2: /VINT -> VBAT
- U1 pad 1: /XL1 -> GND
- U1 pad 10: +3V3 -> unconnected-(U1-P2.01-Pad10)
- U1 pad 16: unconnected-(U1-P2.05/SPI.CS-Pad16) -> GND
- U1 pad 17: unconnected-(U1-P2.06/TRACECLK/SPI.SCK-Pad17) -> /PMIC_INT
- U1 pad 18: /P2.07_SWO -> unconnected-(U1-P0.01-Pad18)
- U1 pad 2: /XL2 -> unconnected-(U1-P2.09-Pad2)
- U1 pad 22: +3V3 -> unconnected-(U1-P1.05-Pad22)
- U1 pad 23: /PMIC_INT -> unconnected-(U1-P1.04-Pad23)
- U1 pad 24: unconnected-(U1-P0.01-Pad24) -> /XL2
- U1 pad 25: /SWDIO -> /XL1
- U1 pad 26: /SWDCLK -> +3V3
- U1 pad 27: unconnected-(U1-P0.02-Pad27) -> GND
- U1 pad 28: unconnected-(U1-P0.03/GRTC_PWMOUT-Pad28) -> /SDA
- U1 pad 30: /NRESET -> unconnected-(U1-P1.08-Pad30)
- U1 pad 31: /ANT -> unconnected-(U1-P0.04-Pad31)
- U1 pad 32: /GND_PA -> unconnected-(U1-P1.14-Pad32)
- U1 pad 33: /DECA -> unconnected-(U1-P1.13-Pad33)
- U1 pad 34: /XC1 -> unconnected-(U1-P1.12-Pad34)
- U1 pad 35: /XC2 -> /SCL
- U1 pad 36: +3V3 -> unconnected-(U1-P0.03-Pad36)
- U1 pad 38: /SDA -> unconnected-(U1-P2.06-Pad38)
- U1 pad 39: /SCL -> GND
- U1 pad 4: unconnected-(U1-P1.03/NFC2-Pad4) -> /P2.07_SWO
- U1 pad 5: unconnected-(U1-P1.04/AIN0/TAMPC-Pad5) -> /SWDIO
- U1 pad 6: unconnected-(U1-P1.05/AIN1/TAMPC-Pad6) -> /SWDCLK
- U1 pad 7: unconnected-(U1-P1.06/AIN2/TAMPC-Pad7) -> /NRESET
- U3 pad 2: /SENSE1 -> /CIN1_PROTECTED
- U3 pad 3: /SENSE2 -> /CIN2_PROTECTED
Routing:
- net /PMIC_INT: track 0.00 -> 57.4 mm, vias 0 -> 2
- net +3V3: track 34.5 -> 63.1 mm, vias 9 -> 4
- net VBAT: track 27.2 -> 1.80 mm
- net /P2.07_SWO: track 10.8 -> 25.0 mm, vias 2 -> 0
- net /SWDCLK: track 13.3 -> 22.4 mm
- net GND: track 15.5 -> 24.5 mm, vias 26 -> 151
- net /SWDIO: track 11.7 -> 20.5 mm
- net /SCL: track 103.8 -> 95.5 mm
- net /DECD: track 6.61 -> 0.00 mm
- net /VINT: track 6.51 -> 0.00 mm
- net /DECA: track 5.55 -> 0.00 mm
- net /NRESET: track 8.19 -> 2.73 mm
- net +3V3_FDC_SW: track 14.6 -> 10.6 mm
- net /XC1: track 3.83 -> 0.00 mm
- net /SWD_RST: track 57.5 -> 61.0 mm
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- added copper zone on F.Cu, net +3V3
- added copper zone on In1.Cu, net /SHLD
- added copper zone on F.Cu, net /VBAT_RAW
- added copper zone on F.Cu, net /VINT
- added copper zone on In2.Cu, net GND
- added copper zone on F.Cu, net VBAT
- removed copper zone on In2.Cu, net +3V3
Other:
- board text added: "A. GOMPPER"
- board text added: "NRF54L15 MOISTURE SENSOR"
- board text added: "REV A 09.05.26"
- board text removed: "SOLAR PRE-REG 8x8 RESERVE"
