File: moisture-sensor-carrier.kicad_sch (KiCad schematic)
At the start: 60 parts, among them J1 USB-C receptacle, J2 Battery - Adafruit 1578, J3 Solar panel, J4 SWD 10p 1.27mm, J5 U.FL-R-SMT-1(10) antenna, U1 nRF54L15-QFAA, U2 nPM1300-QEAA, U3 FDC1004, U4 SHT45-AD1F, U5 TPS7A1650 5V LDO, X1 CM8V-T1A 32.768kHz CL=7pF 20p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, X2 FA-128 32MHz CL=8pF

Commit message: Draw the three chains as chains, not as parts carrying labels
The RF match, the MCU DC/DC and BUCK2 are signal paths, and the order of the
elements is the design. Spelling them as six parts each holding two net labels
gives the same netlist and shows a reader nothing.

  ANT  -> L2 -> L3 -> L4 -> ANT_FEED   with C6, C9, C11 on the nodes between
  DCC  -> L1 -> DECD -> FB1 -> DECA    with C1 on DECD, C2/C12/C5 on DECA
  SW2  -> L10 -> +3V3                  with C24 returning to PVSS2

Nordic draws the first two exactly this way. The DECA bank is the case that
needed it most: DECA and DECRF being one net reads as a mistake until you see
the chain, and three capacitors in a grid each labelled "DECA" is not a bank.
C24's return to PVSS2 rather than to the plane is the whole point of that part
and was previously just a label on its lower pin.

Junctions go 0 -> 8. Text labels 146 -> 84, and what is left is signals.

Supporting changes:

  - place() takes a rotation, and _pin_at() rotates pin anchors to match, so a
    passive can lie flat in a chain. The first attempt emitted rot=0 because
    the f-string patch silently missed; the parts landed correctly and the
    wires missed them, which the netlist fingerprint caught as eight new
    single-pin nets.
  - Chain nodes are named explicitly. KiCad otherwise auto-names them
    Net-(C6-Pad1) - electrically identical, and silently outside every
    netclass pattern and DRU rule keyed on RF_A or RF_B.
  - A node that is a rail gets its rail symbol, not a label. BUCK2's output
    node IS +3V3 and was briefly the one place on the sheet where the 3V3 rail
    did not look like one.
  - Value holds the electrical value; the part number moved to a hidden MPN
    property. "1.5pF GJM0335C1E1R5WB01" is 25 characters hung off a 5 mm
    capacitor and lands on its neighbour. L10 deliberately keeps its
    saturation spec in Value and gets no MPN, because it is specified by
    constraint and does not have one.

The block-overlap g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
Parts:
- C6: value 1.5pF GJM0335C1E1R5WB01 -> 1.5pF; MPN (none) -> GJM0335C1E1R5WB01
- C9: value 2.0pF GJM0335C1E2R0WB01 -> 2.0pF; MPN (none) -> GJM0335C1E2R0WB01
- L1: value MLZ1608M4R7WT000 4.7uH -> 4.7uH; MPN (none) -> MLZ1608M4R7WT000
- L10: value 2.2uH Isat>350mA DCR<400m -> 2.2uH Isat>350mA
- L2: value 2.7nH LQP03HQ2N7B02 -> 2.7nH; MPN (none) -> LQP03HQ2N7B02
- L3, L4: value 3.5nH LQP03HQ3N5B02 -> 3.5nH; MPN (none) -> LQP03HQ3N5B02
