File: nrf-moisture-sensor.kicad_pcb (KiCad board)
At the start: 4 copper layers, 42 x 155 mm, 46 parts, among them J4 SWD 10p 1.27mm, Q1 DMG2305UX-7, U1 453-00001R BL54L15, U2 nPM2100-QEAA, U3 FDC1004, U4 SHT45-AD1F, X1 CM8V-T1A 32.768kHz CL=7pF 20p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

Commit message: Rename nRF Moisture Sensor and review power, pins, schematic and layout
Parts:
- renumbered FID3 to FID4
Routing:
- net GND: track 24.5 -> 25.4 mm, vias 151 -> 154

Commit message: Checkpoint accumulated hardware, bring-up, and manufacturing work
Parts:
- removed FID1, FID2, FID3, FID4: Fiducial, Fiducial:Fiducial_0.5mm_Mask1mm
- added R36, R37: 4.7k 1%, Resistor_SMD:R_0402_1005Metric, F.Cu at (0.00, 0.00)
- added TH1, TH2, TH3: ToolingHole_JLC_1.152mm, footprints:ToolingHole_JLC_1.152mm, F.Cu at (0.00, 0.00)
- added TP10: VINT, TestPoint:TestPoint_Pad_D1.0mm, B.Cu at (0.00, 0.00)
- added TP11, TP5, TP7: GND, TestPoint:TestPoint_Pad_D1.0mm, F.Cu at (0.00, 0.00)
- added TP12: SDA, TestPoint:TestPoint_Pad_D1.0mm, F.Cu at (0.00, 0.00)
- added TP13: SCL, TestPoint:TestPoint_Pad_D1.0mm, F.Cu at (0.00, 0.00)
- added TP14: PMIC_INT, TestPoint:TestPoint_Pad_D1.0mm, F.Cu at (0.00, 0.00)
- added TP15: NRESET, TestPoint:TestPoint_Pad_D1.0mm, F.Cu at (0.00, 0.00)
- added TP16: MARK1, TestPoint:TestPoint_Pad_D1.0mm, F.Cu at (0.00, 0.00)
- added TP17: MARK2, TestPoint:TestPoint_Pad_D1.0mm, F.Cu at (0.00, 0.00)
- added TP4: +3V3, TestPoint:TestPoint_Pad_D1.0mm, F.Cu at (0.00, 0.00)
- added TP6: +3V3_FDC_SW, TestPoint:TestPoint_Pad_D1.0mm, F.Cu at (0.00, 0.00)
- added TP8: VBAT, TestPoint:TestPoint_Pad_D1.0mm, F.Cu at (0.00, 0.00)
- added TP9: VBAT_RAW, TestPoint:TestPoint_Pad_D1.0mm, F.Cu at (0.00, 0.00)
- C21: value 10uF/6.3V X5R -> 22uF/6.3V X5R
- C26: footprint Capacitor_SMD:C_0402_1005Metric_Pad0.74x0.62mm_HandSolder -> Capacitor_SMD:C_0402_1005Metric
- C3: value 10uF/16V X6S -> 10uF/25V X5R
- D1, D10, D2, D3, D4, D5, D6, D7, D8, D9: footprint footprints:TI_DPY0002A -> Package_SON:Texas_DPY0002A_0.6x1mm_P0.65mm
- Q1: value DMG2305UX-7 -> DMG2305UX-13
- R22, R23: value 4.7k to +3V3 -> 4.7k 1%; footprint Resistor_SMD:R_0402_1005Metric_Pad0.72x0.64mm_HandSolder -> Resistor_SMD:R_0402_1005Metric
- U4: value SHT45-AD1F -> SHT40-AD1F
Connections:
- D8 pad 1: /SENSE1 -> /CIN1_PROTECTED
- D9 pad 1: /SENSE2 -> /CIN2_PROTECTED
- U1 pad 20: unconnected-(U1-P1.07-Pad20) -> /MARK1
- U1 pad 21: unconnected-(U1-P1.06-Pad21) -> /MARK2
- U1 pad 22: unconnected-(U1-P1.05-Pad22) -> /FDC_SDA
- U1 pad 23: unconnected-(U1-P1.04-Pad23) -> /FDC_SCL
- U3 pad 10: /SDA -> /FDC_SDA
- U3 pad 9: /SCL -> /FDC_SCL
Routing:
- net /FDC_SDA: track 0.00 -> 61.5 mm, vias 0 -> 4
- net /FDC_SCL: track 0.00 -> 58.3 mm, vias 0 -> 4
- net /SCL: track 95.5 -> 90.3 mm
- net /SDA: track 92.8 -> 87.8 mm
- net GND: track 25.4 -> 23.4 mm, vias 154 -> 329
- net /MARK1: track 0.00 -> 1.98 mm
- net +3V3: track 63.1 -> 64.9 mm
- net /MARK2: track 0.00 -> 1.74 mm
- net /PMIC_INT: track 57.4 -> 59.0 mm
- net /SHLD: track 1.09 -> 2.46 mm, vias 105 -> 113
- net /NRESET: track 2.73 -> 4.01 mm
- net /CIN1_PROTECTED: track 1.45 -> 2.17 mm
- net /CIN2_PROTECTED: track 1.70 -> 2.39 mm
- net +3V3_FDC_SW: track 10.6 -> 9.97 mm
- net /VINT: track 0.00 -> 0.59 mm, vias 0 -> 1
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- added copper zone on B.Cu, net /SENSE1
- added copper zone on In1.Cu, net /SENSE1
- added copper zone on In2.Cu, net /SENSE1
- added copper zone on B.Cu, net /SENSE2
- added copper zone on In1.Cu, net /SENSE2
- added copper zone on In2.Cu, net /SENSE2
Other:
- outline, holes or cut-outs redrawn
- board text added: "3V3"
- board text added: "FDC"
- board text added: "GND"
- board text added: "INT"
- board text added: "M1"
- board text added: "M2"
- board text added: "RAW"
- board text added: "RST"
- board text added: "SCL"
- board text added: "SDA"
- board text added: "VBAT"
- board text added: "VINT"

Commit message: Checkpoint Rev A consolidated BOM and JLC-reviewed fabrication baseline
Parts:
- removed C13: 3.9pF C0G, Capacitor_SMD:C_0402_1005Metric
- removed R1: 1k 1%, Resistor_SMD:R_0402_1005Metric
- C21, C23: value 22uF/6.3V X5R -> 10uF/25V X5R; footprint Capacitor_SMD:C_0402_1005Metric -> Capacitor_SMD:C_0603_1608Metric
- C26: value 1uF 10V X7R -> 2.2uF/6.3V X5R
- D1, D2, D3: value TPD1E1B04DPYR -> TPD1E01B04DPYR
- R30, R31: value 5.1k 1% -> 4.7k 1%
- U4: value SHT40-AD1F -> SHT40-AD1B
Connections:
- R35 pad 2: /SWD_RST -> /NRESET
- U2 pad 10: /SWD_RST -> /NRESET
Routing:
- net /SWD_RST: track 60.5 -> 0.00 mm, vias 2 -> 0
- net /NRESET: track 4.01 -> 63.7 mm, vias 0 -> 2
- net GND: vias 329 -> 330
