File: nrf-moisture-sensor.kicad_sch (KiCad schematic)
At the start: 44 parts, among them J4 SWD 10p 1.27mm, Q1 DMG2305UX-7, U1 453-00001R BL54L15, U2 nPM2100-QEAA, U3 FDC1004, U4 SHT45-AD1F, X1 CM8V-T1A 32.768kHz CL=7pF 20p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

Commit message: Checkpoint accumulated hardware, bring-up, and manufacturing work
Parts:
- removed FID1, FID2, FID3: Fiducial, Fiducial:Fiducial_0.5mm_Mask1mm, symbol Mechanical:Fiducial
- added R36, R37: 4.7k 1%, Resistor_SMD:R_0402_1005Metric, symbol Device:R_Small_US
- added TP10: VINT, TestPoint:TestPoint_Pad_D1.0mm, symbol Connector:TestPoint
- added TP11, TP5, TP7: GND, TestPoint:TestPoint_Pad_D1.0mm, symbol Connector:TestPoint
- added TP12: SDA, TestPoint:TestPoint_Pad_D1.0mm, symbol Connector:TestPoint
- added TP13: SCL, TestPoint:TestPoint_Pad_D1.0mm, symbol Connector:TestPoint
- added TP14: PMIC_INT, TestPoint:TestPoint_Pad_D1.0mm, symbol Connector:TestPoint
- added TP15: NRESET, TestPoint:TestPoint_Pad_D1.0mm, symbol Connector:TestPoint
- added TP16: MARK1, TestPoint:TestPoint_Pad_D1.0mm, symbol Connector:TestPoint
- added TP17: MARK2, TestPoint:TestPoint_Pad_D1.0mm, symbol Connector:TestPoint
- added TP4: +3V3, TestPoint:TestPoint_Pad_D1.0mm, symbol Connector:TestPoint
- added TP6: +3V3_FDC_SW, TestPoint:TestPoint_Pad_D1.0mm, symbol Connector:TestPoint
- added TP8: VBAT, TestPoint:TestPoint_Pad_D1.0mm, symbol Connector:TestPoint
- added TP9: VBAT_RAW, TestPoint:TestPoint_Pad_D1.0mm, symbol Connector:TestPoint
- C21: value 10uF/6.3V X5R -> 22uF/6.3V X5R; LCSC C15525 -> C3894351; MPN CL05A106MQ5NUNC -> GRM158R60J226ME01D; Manufacturer Samsung -> Murata Electronics
- C23: LCSC C415703 -> C3894351; MPN GRM155R60J226ME11D -> GRM158R60J226ME01D; Manufacturer Murata -> Murata Electronics
- C26: footprint Capacitor_SMD:C_0402_1005Metric_Pad0.74x0.62mm_HandSolder -> Capacitor_SMD:C_0402_1005Metric
- C3: value 10uF/16V X6S -> 10uF/25V X5R; LCSC C3039688 -> C96446; MPN CL10X106MO8NRNC -> CL10A106MA8NRNC
- D1, D10, D2, D3, D4, D5, D6, D7, D8, D9: footprint footprints:TI_DPY0002A -> Package_SON:Texas_DPY0002A_0.6x1mm_P0.65mm
- Q1: value DMG2305UX-7 -> DMG2305UX-13; LCSC C150470 -> C144153; MPN DMG2305UX-7 -> DMG2305UX-13
- R22, R23: value 4.7k to +3V3 -> 4.7k 1%; footprint Resistor_SMD:R_0402_1005Metric_Pad0.72x0.64mm_HandSolder -> Resistor_SMD:R_0402_1005Metric
- U4: value SHT45-AD1F -> SHT40-AD1F; LCSC C5360602 -> C7461846; MPN SHT45-AD1F-R2 -> SHT40-AD1F-R2
Connections:
- net +3V3: now also TP4.1
- net +3V3_FDC_SW: now also R36.1, R37.1, TP6.1
- net CIN1_PROTECTED: now also D8.1 (A1)
- net CIN2_PROTECTED: now also D9.1 (A1)
- net GND: now also TP11.1, TP5.1, TP7.1
- net NRESET: now also TP15.1
- net PMIC_INT: now also TP14.1
- net SCL: now also TP13.1; no longer U3.9 (SCL)
- net SDA: now also TP12.1; no longer U3.10 (SDA)
- net SENSE1: no longer D8.1 (A1)
- net SENSE2: no longer D9.1 (A1)
- net VBAT: now also TP8.1
- net VBAT_RAW: now also TP9.1
- net VINT: now also TP10.1
- net MARK1: now reaches U1.20 (P1.07)
- net MARK1: now also TP16.1
- net MARK2: now reaches U1.21 (P1.06)
- net MARK2: now also TP17.1
- net FDC_SDA: now reaches U1.22 (P1.05)
- net FDC_SDA: now also U3.10 (SDA), R36.2
- net FDC_SCL: now reaches U1.23 (P1.04)
- net FDC_SCL: now also U3.9 (SCL), R37.2
- no-connect marks 34 -> 30
Other:
- note added: "FDC1004: switched supply. SHT40: main +3V3 supply."
- note removed: "FDC1004: switched supply. SHT45: main +3V3 supply."

Commit message: Checkpoint Rev A consolidated BOM and JLC-reviewed fabrication baseline
Parts:
- removed C13: 3.9pF C0G, Capacitor_SMD:C_0402_1005Metric, symbol Device:C_Small
- removed R1: 1k 1%, Resistor_SMD:R_0402_1005Metric, symbol Device:R_Small
- C21, C23: value 22uF/6.3V X5R -> 10uF/25V X5R; footprint Capacitor_SMD:C_0402_1005Metric -> Capacitor_SMD:C_0603_1608Metric; LCSC C3894351 -> C96446; MPN GRM158R60J226ME01D -> CL10A106MA8NRNC; Manufacturer Murata Electronics -> Samsung
- C26: value 1uF 10V X7R -> 2.2uF/6.3V X5R; LCSC C528974 -> C12530; MPN GRM155Z71A105KE01D -> CL05A225MQ5NSNC; Manufacturer Murata -> Samsung
- D1, D2, D3: value TPD1E1B04DPYR -> TPD1E01B04DPYR; symbol protection:TPD1E1B04 -> protection:TPD1E01B04; LCSC C779408 -> C779389; MPN TPD1E1B04DPYR -> TPD1E01B04DPYR
- R30, R31: value 5.1k 1% -> 4.7k 1%; LCSC C25905 -> C25900; MPN 0402WGF5101TCE -> 0402WGF4701TCE
- U4: value SHT40-AD1F -> SHT40-AD1B; LCSC C7461846 -> C2909890; MPN SHT40-AD1F-R2 -> SHT40-AD1B-R2
Connections:
- net SWD_RST is gone; now on net NRESET: R35.2, U2.10 (PG/RESET)
Other:
- note added: "CIN1 / CIN2 via 4.7k protection; SHLD driven by FDC."
- note added: "Reset: direct host / PMIC connection."
- note removed: "CIN1 / CIN2 via 5.1k protection; SHLD driven by FDC."
- note removed: "R1 / C13: module reset input network."
